File: OSBAMS_Pi_Display_Power_RevA_RC1/kicad/OSBAMS_Pi_Display_Power_RevA.kicad_sch (KiCad schematic)
At the start: 18 parts, among them U1 RSDW40F-05

Commit message: Pi/Display power board RC1.1: library footprints, 5V drop budget, DNP trim pads
Replace hand-drawn footprints with official KiCad ones (fixes Micro-Fit
row numbering and Nano2 size), re-lay the 5V path, add voltage-drop budget
script/doc, 16 AWG/150 mm harness, DNP trim network. RSDW40F-05 footprint is
still an unverified placeholder; RC2 intentionally not generated.

Co-Authored-By: Claude Sonnet 5.5 <noreply@anthropic.com>
Claude-Session: https://claude.ai/code/session_01ENatZXrEDA18PaxUrZWrpi
Parts:
- added R2: DNP, Resistor_SMD:R_0603_1608Metric, symbol OSBAMS_PiPwr:R2
- added R3: DNP, Resistor_SMD:R_0603_1608Metric, symbol OSBAMS_PiPwr:R3
- C1, C6: footprint OSBAMS_PiPwr:C0603 -> Capacitor_SMD:C_0603_1608Metric
- C2: footprint OSBAMS_PiPwr:CP_RADIAL_D8_P35 -> Capacitor_THT:CP_Radial_D8.0mm_P3.50mm
- C4: footprint OSBAMS_PiPwr:CP_RADIAL_D10_P50 -> Capacitor_THT:CP_Radial_D10.0mm_P5.00mm
- C5: footprint OSBAMS_PiPwr:C0805 -> Capacitor_SMD:C_0805_2012Metric
- D1: footprint OSBAMS_PiPwr:LED0603 -> LED_SMD:LED_0603_1608Metric
- F1: footprint OSBAMS_PiPwr:FUSE_NANO2_H -> Fuse:Fuse_Littelfuse-NANO2-451_453
- F2: footprint OSBAMS_PiPwr:FUSE_NANO2_V -> Fuse:Fuse_Littelfuse-NANO2-451_453
- J_IN: footprint OSBAMS_PiPwr:MICROFIT_RA_2 -> Connector_Molex:Molex_Micro-Fit_3.0_43045-0200_2x01_P3.00mm_Horizontal
- J_OUT: footprint OSBAMS_PiPwr:MICROFIT_RA_4 -> Connector_Molex:Molex_Micro-Fit_3.0_43045-0400_2x02_P3.00mm_Horizontal
- R1: footprint OSBAMS_PiPwr:R0603 -> Resistor_SMD:R_0603_1608Metric
- TP1, TP2, TP3, TP4, TP5: footprint OSBAMS_PiPwr:TP15 -> TestPoint:TestPoint_Pad_D1.5mm
- TVS1: footprint OSBAMS_PiPwr:DO214AA -> Diode_SMD:D_SMB
- U1: footprint OSBAMS_PiPwr:RSDW40_PLACEHOLDER -> OSBAMS_PiPwr:RSDW40F-05_PLACEHOLDER_UNVERIFIED
Connections:
- net 5V_ISO_RAW: now also R2.2
- net 5V_PI: now also C5.1, C6.1; no longer C5.2, C6.2
- net PI_GND: now also C5.2, C6.2, R3.2; no longer C5.1, C6.1
- net TRIM: now reaches U1.6 (TRIM)
- net TRIM: now also R2.1, R3.1
- no-connect marks 2 -> 1
Other:
- note added: "U1 pin 3 (ON/OFF) left open - confirm default state. TRIM (pin 6) only goes to DNP pads R2/R3 (do not fit without Mean Well trim formula)."
- note removed: "U1 pin 3 (ON/OFF) and pin 6 (TRIM) intentionally unconnected - confirm remote ON/OFF default state vs Mean Well datasheet."

Commit message: Keyed Pi interposer, F1 8A time-delay, calibration procedure, budget update
Add OSBAMS_Pi_Power_Interposer_RevA_RC1 (Micro-Fit + 2x20 stacking socket, key
standoffs), trim calibration script/procedure/acceptance record, F1 candidate
0453008.MRL, budget with interposer path. RC2 still gated: F1 datasheet,
socket MPN, key 3D check, KiCad 10 ERC.

Co-Authored-By: Claude Sonnet 5.5 <noreply@anthropic.com>
Claude-Session: https://claude.ai/code/session_01ENatZXrEDA18PaxUrZWrpi
Parts:
- F1: value 5A 125V -> 8A 125V TD; MPN 0451005.MRL -> 0453008.MRL
Changed lines of the file:
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@@
 (symbol (lib_id "OSBAMS_PiPwr:F1") (at 71.12 38.10 0) (unit 1) (in_bom yes) (on_board yes) (dnp no)
   (property "Reference" "F1" (at 71.12 32.10 0) (effects (font (size 1.27 1.27))))
-  (property "Value" "5A 125V" (at 71.12 44.10 0) (effects (font (size 1.27 1.27))))
+  (property "Value" "8A 125V TD" (at 71.12 44.10 0) (effects (font (size 1.27 1.27))))
   (property "Footprint" "Fuse:Fuse_Littelfuse-NANO2-451_453" (at 71.12 38.10 0) (effects (font (size 1.27 1.27)) hide))
   (property "Datasheet" "" (at 71.12 38.10 0) (effects hide))
   (property "Manufacturer" "Littelfuse" (at 71.12 38.10 0) (effects hide))
-  (property "MPN" "0451005.MRL" (at 71.12 38.10 0) (effects hide))
+  (property "MPN" "0453008.MRL" (at 71.12 38.10 0) (effects hide))
   (pin "1")(pin "2")
   (instances (project "OSBAMS_Pi_Display_Power_RevA" (path "/7f3c1a52-0d4e-4c8e-9b61-5a0e3f2d1c11" (reference "F1") (unit 1)))))

Commit message: F1 -> Littelfuse 407 8A time-lag (0407008.WR); F2 verified; interposer to HAT+ geometry
Remove 0453008.MRL (very fast-acting). F1 datasheet values and 1206 land pattern
implemented; F2 footprint verified against 451/453 datasheet. Interposer now 65 mm
with M2.5 mounting holes per HAT+ spec. RC2 still gated: socket MPN, Pi 5 STEP
keying check, KiCad 10 ERC.

Co-Authored-By: Claude Sonnet 5.5 <noreply@anthropic.com>
Claude-Session: https://claude.ai/code/session_01ENatZXrEDA18PaxUrZWrpi
Parts:
- F1: value 8A 125V TD -> 8A TIME-LAG 24V; footprint Fuse:Fuse_Littelfuse-NANO2-451_453 -> OSBAMS_PiPwr:Fuse_1206_Littelfuse407; MPN 0453008.MRL -> 0407008.WR
- U1: footprint OSBAMS_PiPwr:RSDW40F-05_PLACEHOLDER_UNVERIFIED -> OSBAMS_PiPwr:RSDW40F-05_MeanWell_2x1in
Changed lines of the file:
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@@
 (symbol (lib_id "OSBAMS_PiPwr:F1") (at 71.12 38.10 0) (unit 1) (in_bom yes) (on_board yes) (dnp no)
   (property "Reference" "F1" (at 71.12 32.10 0) (effects (font (size 1.27 1.27))))
-  (property "Value" "8A 125V TD" (at 71.12 44.10 0) (effects (font (size 1.27 1.27))))
-  (property "Footprint" "Fuse:Fuse_Littelfuse-NANO2-451_453" (at 71.12 38.10 0) (effects (font (size 1.27 1.27)) hide))
+  (property "Value" "8A TIME-LAG 24V" (at 71.12 44.10 0) (effects (font (size 1.27 1.27))))
+  (property "Footprint" "OSBAMS_PiPwr:Fuse_1206_Littelfuse407" (at 71.12 38.10 0) (effects (font (size 1.27 1.27)) hide))
   (property "Datasheet" "" (at 71.12 38.10 0) (effects hide))
   (property "Manufacturer" "Littelfuse" (at 71.12 38.10 0) (effects hide))
-  (property "MPN" "0453008.MRL" (at 71.12 38.10 0) (effects hide))
+  (property "MPN" "0407008.WR" (at 71.12 38.10 0) (effects hide))
   (pin "1")(pin "2")
   (instances (project "OSBAMS_Pi_Display_Power_RevA" (path "/7f3c1a52-0d4e-4c8e-9b61-5a0e3f2d1c11" (reference "F1") (unit 1)))))
@@
   (property "Reference" "U1" (at 116.84 108.30 0) (effects (font (size 1.27 1.27))))
   (property "Value" "RSDW40F-05" (at 116.84 120.30 0) (effects (font (size 1.27 1.27))))
-  (property "Footprint" "OSBAMS_PiPwr:RSDW40F-05_PLACEHOLDER_UNVERIFIED" (at 116.84 114.30 0) (effects (font (size 1.27 1.27)) hide))
+  (property "Footprint" "OSBAMS_PiPwr:RSDW40F-05_MeanWell_2x1in" (at 116.84 114.30 0) (effects (font (size 1.27 1.27)) hide))
   (property "Datasheet" "" (at 116.84 114.30 0) (effects hide))
   (property "Manufacturer" "Mean Well" (at 116.84 114.30 0) (effects hide))
