File: Hardware/Rev2_Controller/OSBAMS_Rev2_RELEASE_CANDIDATE_1/01_Power_Input.kicad_sch (KiCad schematic)
At the start: 5 parts, among them J1 12V_IN

Commit message: RC1: EB21A-02-C footprint verified against the Adam Tech drawing (rev B); J1-J4 re-placed, board re-routed
Hole 1.30 mm, body 10.6 x 8.5 mm, wire entry toward the board edge; VERIFY_MECHANICAL_DRAWING removed
for this part only. ERC 0; DRC: 0 electrical, 4 silkscreen warnings, 0 unconnected.

Co-Authored-By: Claude Sonnet 5.5 <noreply@anthropic.com>
Claude-Session: https://claude.ai/code/session_01HV1TCrYnLTcNjmYdFqCPLo
Parts:
- J1: footprint OSBAMS_Rev2:EB21A-02-C_PROVISIONAL -> OSBAMS_Rev2:EB21A-02-C
