File: Hardware/Rev2_Controller/OSBAMS_Rev2_RELEASE_CANDIDATE_1/02_Buck_3V3.kicad_sch (KiCad schematic)
At the start: 16 parts, among them U3 LMR14006Y

Commit message: RC1.1: ISO7721 pinout fix, CP2102N VBUS divider/RSTb pull-up/VDD bypass, datasheets read locally
- ISO7721 symbol corrected to the TI D/DWV table (2 OUTA, 3 INB, 6 OUTB, 7 INA); UART nets reassigned and re-routed
- CP2102N: VBUS 22.1k/47.5k divider (R38/R39), 1k RSTb pull-up (R40), VDD bypass 4.7uF (C22) per the datasheet
- ISO7721, CP2102N, SRN6045TA datasheets committed as evidence and marked VERIFIED_LOCAL; SRN6045TA-100M inductor closed
- isolation check script/report (3.0 mm in the ISO7721 area, 0.25 mm elsewhere); docs corrected (netclass clearances)
- board re-placed and re-routed: ERC 0, DRC 0 electrical (3 silkscreen warnings), netlist 0 mismatches

Co-Authored-By: Claude Sonnet 5.5 <noreply@anthropic.com>
Claude-Session: https://claude.ai/code/session_01HV1TCrYnLTcNjmYdFqCPLo
Parts:
- L1: Evidence UNVERIFIED -> VERIFIED_LOCAL
