File: Hardware/Rev2_Controller/OSBAMS_Rev2_RELEASE_CANDIDATE_1/03_MCU.kicad_sch (KiCad schematic)
At the start: 16 parts, among them J9 SWD, SW1 RESET, U1 STM32L476RGT6

Commit message: RC1: reconcile user-relayed manufacturer data (USER_RELAYED_MANUFACTURER)
- audit report MANUFACTURER_DATA_RECONCILIATION.md; INA228/STM32/IRLML0060/LMR14006Y/CP2102N/VO610A/TC74 pin maps match the relayed data
- ISO7721 pin-direction conflict left unresolved (needs the TI pin diagram); CP2102N VBUS reference connection open
- LMR14006Y: 95 ns TON_MIN analysis (15 V marginal, 24.4 V below TON_MIN); 1.5SMBJ48A vs INA228 85 V clamp-vs-current analysis
- firmware: INA228 IMAX 30 A -> 20 A (SHUNT_CAL 1250) + test
- fix: TC74 probe PCB had been left unrouted by the schematic step; re-routed, DRC 0; schematic step no longer rebuilds it

Co-Authored-By: Claude Sonnet 5.5 <noreply@anthropic.com>
Claude-Session: https://claude.ai/code/session_01HV1TCrYnLTcNjmYdFqCPLo
Parts:
- U1: Evidence UNVERIFIED -> USER_RELAYED_MANUFACTURER

Commit message: RC1.2e: Samtec J9 land pattern (0.74x2.79, rev H), D15 differential clamp across INA228 IN+/IN-, protection and connector audit; ERJ-P08 pulse capability re-opened
- J9 generic footprint replaced by OSBAMS_Rev2:FTSH-105-01-L-DV-K from the Samtec recommended layout rev H; breakout re-routed
- D15 SMF12CA bidirectional TVS across INA_INP/INA_INN (INA228 differential limit +/-40 V; one Kelvin lead open)
- CONTROLLER_PROTECTION_AND_CONNECTOR_AUDIT.md (PASS / CHANGE REQUIRED / FIRST-ARTICLE VALIDATION / REMAINING FABRICATION BLOCKERS)
- rs_pulse_rating back to UNVERIFIED/critical; Molex J5/J6 stay open (3D drawing without dimensions); evidence PDFs committed
- ERC 0, DRC 0, unconnected 0, netlist 0 mismatches (405 pads), polarity OK, isolation >= 1.0 mm; 181 tests pass

Co-Authored-By: Claude Sonnet 5.5 <noreply@anthropic.com>
Claude-Session: https://claude.ai/code/session_01HV1TCrYnLTcNjmYdFqCPLo
Parts:
- J9: footprint Connector_PinHeader_1.27mm:PinHeader_2x05_P1.27mm_Vertical_SMD -> OSBAMS_Rev2:FTSH-105-01-L-DV-K
