File: Hardware/Rev2_Controller/OSBAMS_Rev2_RELEASE_CANDIDATE_1/04_Host_Isolated.kicad_sch (KiCad schematic)
At the start: 14 parts, among them J8 USB-C HOST, U6 CP2102N, U7 ISO7721, U9 USBLC6-2SC6

Commit message: RC1: reconcile user-relayed manufacturer data (USER_RELAYED_MANUFACTURER)
- audit report MANUFACTURER_DATA_RECONCILIATION.md; INA228/STM32/IRLML0060/LMR14006Y/CP2102N/VO610A/TC74 pin maps match the relayed data
- ISO7721 pin-direction conflict left unresolved (needs the TI pin diagram); CP2102N VBUS reference connection open
- LMR14006Y: 95 ns TON_MIN analysis (15 V marginal, 24.4 V below TON_MIN); 1.5SMBJ48A vs INA228 85 V clamp-vs-current analysis
- firmware: INA228 IMAX 30 A -> 20 A (SHUNT_CAL 1250) + test
- fix: TC74 probe PCB had been left unrouted by the schematic step; re-routed, DRC 0; schematic step no longer rebuilds it

Co-Authored-By: Claude Sonnet 5.5 <noreply@anthropic.com>
Claude-Session: https://claude.ai/code/session_01HV1TCrYnLTcNjmYdFqCPLo
Parts:
- U6: Evidence UNVERIFIED -> USER_RELAYED_MANUFACTURER
- U7: Evidence USER_RELAYED_MANUFACTURER -> UNVERIFIED

Commit message: RC1.1: ISO7721 pinout fix, CP2102N VBUS divider/RSTb pull-up/VDD bypass, datasheets read locally
- ISO7721 symbol corrected to the TI D/DWV table (2 OUTA, 3 INB, 6 OUTB, 7 INA); UART nets reassigned and re-routed
- CP2102N: VBUS 22.1k/47.5k divider (R38/R39), 1k RSTb pull-up (R40), VDD bypass 4.7uF (C22) per the datasheet
- ISO7721, CP2102N, SRN6045TA datasheets committed as evidence and marked VERIFIED_LOCAL; SRN6045TA-100M inductor closed
- isolation check script/report (3.0 mm in the ISO7721 area, 0.25 mm elsewhere); docs corrected (netclass clearances)
- board re-placed and re-routed: ERC 0, DRC 0 electrical (3 silkscreen warnings), netlist 0 mismatches

Co-Authored-By: Claude Sonnet 5.5 <noreply@anthropic.com>
Claude-Session: https://claude.ai/code/session_01HV1TCrYnLTcNjmYdFqCPLo
Parts:
- added R38: 22.1k, Resistor_SMD:R_0603_1608Metric, symbol Device:R
- added R39: 47.5k, Resistor_SMD:R_0603_1608Metric, symbol Device:R
- added R40: 1k, Resistor_SMD:R_0603_1608Metric, symbol Device:R
- C22: value 1uF -> 4.7uF; Alternate Samsung CL21B105KOFNNNE -> Samsung CL21A475KPFNNNE; MPN GRM21BR71C105KA01L -> GRM21BR61A475KA73L; Note (none) -> CP2102N VDD: 4.7 uF + 0.1 uF required per power pin (Silico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
- U6: Evidence USER_RELAYED_MANUFACTURER -> VERIFIED_LOCAL
- U7: Evidence UNVERIFIED -> VERIFIED_LOCAL; Note (none) -> Channel A (INA pin 7, host side) -> OUTA pin 2 (MCU RX); ch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
Connections:
- net 3V3_HOST: now also R40.2
- net GND_HOST: now also R39.2
- net UART_RX_HOST: now also U7.6 (OUTB); no longer U7.7 (OUTA)
- net UART_RX_MCU: now also U7.2 (OUTA); no longer U7.3 (OUTB)
- net UART_TX_HOST: now also U7.7 (INA); no longer U7.6 (INB)
- net UART_TX_MCU: now also U7.3 (INB); no longer U7.2 (INA)
- net VBUS_USB: now also R38.1; no longer U6.8 (VBUS)
- net CP_RSTB: now reaches U6.9 (~{RST})
- net CP_RSTB: now also R40.1
- new net CP_VBUS_SENSE: R38.2, R39.1, U6.8 (VBUS)
- no-connect marks 13 -> 12

Commit message: RC1.2: CP2102N VBUS divider margin (R38 19.1k), protection marked not fully closed, isolation-rule activity check
- R38 22.1k -> 19.1k from the CP2102N datasheet limits (VIH = VDD-0.6 V; +0.12 V at VBUS 4.40 V / VDD 3.6 V / 1 %); value change only, layout unchanged
- pack-sense protection: model PASS but not closed (ERJ-P08F pulse rating, 1.5SMBJ48A leakage unread); surge-capability numbers labelled model results
- ISOLATION_RULE_CHECK: the .kicad_dru is applied from a fresh folder; pack-net rule documented as a low-voltage sense-net rule
- connector drawings still not available: footprints unchanged, item open
- ERC 0, DRC 0, unconnected 0, netlist 0 mismatches, polarity none; no Gerbers in the package

Co-Authored-By: Claude Sonnet 5.5 <noreply@anthropic.com>
Claude-Session: https://claude.ai/code/session_01HV1TCrYnLTcNjmYdFqCPLo
Parts:
- R38: value 22.1k -> 19.1k; MPN CRCW060322K1FKEA -> CRCW060319K1FKEA; Note CP2102N VBUS sense divider (Silicon Labs reference, relayed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 -> CP2102N VBUS sense divider upper resistor: Silicon Labs ref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
- R39: Note CP2102N VBUS sense divider: 47.5 k lower -> CP2102N VBUS sense divider lower resistor (Silicon Labs ref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
