File: Hardware/Rev2_Controller/OSBAMS_Rev2_RELEASE_CANDIDATE_1/07_Coil_Driver.kicad_sch (KiCad schematic)
At the start: 9 parts, among them J2 ESTOP, J3 ARM, J4 K1_COIL, Q1 IRLML0060

Commit message: RC1: EB21A-02-C footprint verified against the Adam Tech drawing (rev B); J1-J4 re-placed, board re-routed
Hole 1.30 mm, body 10.6 x 8.5 mm, wire entry toward the board edge; VERIFY_MECHANICAL_DRAWING removed
for this part only. ERC 0; DRC: 0 electrical, 4 silkscreen warnings, 0 unconnected.

Co-Authored-By: Claude Sonnet 5.5 <noreply@anthropic.com>
Claude-Session: https://claude.ai/code/session_01HV1TCrYnLTcNjmYdFqCPLo
Parts:
- J2, J3, J4: footprint OSBAMS_Rev2:EB21A-02-C_PROVISIONAL -> OSBAMS_Rev2:EB21A-02-C

Commit message: RC1: reconcile user-relayed manufacturer data (USER_RELAYED_MANUFACTURER)
- audit report MANUFACTURER_DATA_RECONCILIATION.md; INA228/STM32/IRLML0060/LMR14006Y/CP2102N/VO610A/TC74 pin maps match the relayed data
- ISO7721 pin-direction conflict left unresolved (needs the TI pin diagram); CP2102N VBUS reference connection open
- LMR14006Y: 95 ns TON_MIN analysis (15 V marginal, 24.4 V below TON_MIN); 1.5SMBJ48A vs INA228 85 V clamp-vs-current analysis
- firmware: INA228 IMAX 30 A -> 20 A (SHUNT_CAL 1250) + test
- fix: TC74 probe PCB had been left unrouted by the schematic step; re-routed, DRC 0; schematic step no longer rebuilds it

Co-Authored-By: Claude Sonnet 5.5 <noreply@anthropic.com>
Claude-Session: https://claude.ai/code/session_01HV1TCrYnLTcNjmYdFqCPLo
Parts:
- Q1: Evidence UNVERIFIED -> USER_RELAYED_MANUFACTURER
