File: Hardware/Rev2_Controller/OSBAMS_Rev2_RELEASE_CANDIDATE_1/OSBAMS_Rev2_RC1.kicad_pcb (KiCad board)
At the start: 4 copper layers, 100 x 90 mm, 149 parts, among them J1 12V_IN, J2 ESTOP, J3 ARM, J4 K1_COIL, J5 SHUNT_KELVIN, J6 PACK_SENSE, J7 TEMP_PROBE, J8 USB-C HOST, J9 SWD, Q1 IRLML0060, SW1 RESET, U1 STM32L476RGT6, U10 USBLC6-2SC6, U2 INA228, U3 LMR14006Y, U4 VO610A-1, U5 VO610A-1, U6 CP2102N, U7 ISO7721, U9 USBLC6-2SC6

Commit message: RC1.2e: PCB net names and footprint fields now identical to the schematic (KiCad schematic-parity DRC = 0); fixes ~1370 DRC violations after 'Update PCB from Schematic'; HOST domain/isolation rules and checks made name-form independent; geometry unchanged
Co-Authored-By: Claude Sonnet 5.5 <noreply@anthropic.com>
Claude-Session: https://claude.ai/code/session_01HV1TCrYnLTcNjmYdFqCPLo
Connections:
- net 12V_F renamed /01_Power_Input/12V_F
- net 12V_RAW renamed /01_Power_Input/12V_RAW
- net ADC_MID renamed /06_ADC_PackSense/ADC_MID
- net ADC_TAP renamed /06_ADC_PackSense/ADC_TAP
- net ARM_DIV renamed /08_Status_Sense/ARM_DIV
- net BOOT0 renamed /03_MCU/BOOT0
- net BUCK_CB renamed /02_Buck_3V3/BUCK_CB
- net BUCK_EN renamed /02_Buck_3V3/BUCK_EN
- net BUCK_FB renamed /02_Buck_3V3/BUCK_FB
- net BUCK_SW renamed /02_Buck_3V3/BUCK_SW
- net CP_RSTB renamed /04_Host_Isolated/CP_RSTB
- net CP_VBUS_SENSE renamed /04_Host_Isolated/CP_VBUS_SENSE
- net ES_LED_A renamed /08_Status_Sense/ES_LED_A
- net FB_LED_A renamed /08_Status_Sense/FB_LED_A
- net FB_R1 renamed /08_Status_Sense/FB_R1
- net FB_R2 renamed /08_Status_Sense/FB_R2
- net LED_3V3 renamed /02_Buck_3V3/LED_3V3
- net LED_COIL renamed /07_Coil_Driver/LED_COIL
- net LED_HB renamed /03_MCU/LED_HB
- net LED_HB_PIN renamed /03_MCU/LED_HB_PIN
- net PACK_ADC renamed /06_ADC_PackSense/PACK_ADC
- net PACK_INA renamed /05_INA228_Shunt/PACK_INA
- net SCL2_J renamed /09_Temp_Probe/SCL2_J
- net SCL2_P renamed /09_Temp_Probe/SCL2_P
- net SDA2_J renamed /09_Temp_Probe/SDA2_J
- net SDA2_P renamed /09_Temp_Probe/SDA2_P
- net SHUNT_INN_CON renamed /05_INA228_Shunt/SHUNT_INN_CON
- net SHUNT_INN_RAW renamed /05_INA228_Shunt/SHUNT_INN_RAW
- net SHUNT_INP_CON renamed /05_INA228_Shunt/SHUNT_INP_CON
- net SHUNT_INP_RAW renamed /05_INA228_Shunt/SHUNT_INP_RAW
- net SWO renamed /03_MCU/SWO
- net UART_RX_HOST renamed /04_Host_Isolated/UART_RX_HOST
- net UART_TX_HOST renamed /04_Host_Isolated/UART_TX_HOST
- net USB_CC1 renamed /04_Host_Isolated/USB_CC1
- net USB_CC2 renamed /04_Host_Isolated/USB_CC2
- net USB_DM renamed /04_Host_Isolated/USB_DM
- net USB_DM_J renamed /04_Host_Isolated/USB_DM_J
- net USB_DP renamed /04_Host_Isolated/USB_DP
- net USB_DP_J renamed /04_Host_Isolated/USB_DP_J
- net USB_SHIELD renamed /04_Host_Isolated/USB_SHIELD
- net VCLAMP renamed /06_ADC_PackSense/VCLAMP
- D14 pad 2: (no net) -> unconnected-(D14-K-Pad2)
- J8 pad A8: (no net) -> unconnected-(J8-SBU1-PadA8)
- J8 pad B8: (no net) -> unconnected-(J8-SBU2-PadB8)
- J9 pad 7: (no net) -> unconnected-(J9-KEY-Pad7)
- J9 pad 8: (no net) -> unconnected-(J9-NC/TDI-Pad8)
- U1 pad 10: (no net) -> unconnected-(U1-PC2-Pad10)
- U1 pad 11: (no net) -> unconnected-(U1-PC3-Pad11)
- U1 pad 2: (no net) -> unconnected-(U1-PC13-Pad2)
- U1 pad 20: (no net) -> unconnected-(U1-PA4-Pad20)
- U1 pad 22: (no net) -> unconnected-(U1-PA6-Pad22)
- U1 pad 23: (no net) -> unconnected-(U1-PA7-Pad23)
- U1 pad 24: (no net) -> unconnected-(U1-PC4-Pad24)
- U1 pad 25: (no net) -> unconnected-(U1-PC5-Pad25)
- U1 pad 27: (no net) -> unconnected-(U1-PB1-Pad27)
- U1 pad 28: (no net) -> unconnected-(U1-PB2-Pad28)
- U1 pad 3: (no net) -> unconnected-(U1-PC14-Pad3)
- U1 pad 33: (no net) -> unconnected-(U1-PB12-Pad33)
- U1 pad 34: (no net) -> unconnected-(U1-PB13-Pad34)
- U1 pad 35: (no net) -> unconnected-(U1-PB14-Pad35)
- U1 pad 36: (no net) -> unconnected-(U1-PB15-Pad36)
- U1 pad 37: (no net) -> unconnected-(U1-PC6-Pad37)
- U1 pad 38: (no net) -> unconnected-(U1-PC7-Pad38)
- U1 pad 4: (no net) -> unconnected-(U1-PC15-Pad4)
- U1 pad 41: (no net) -> unconnected-(U1-PA8-Pad41)
- U1 pad 42: (no net) -> unconnected-(U1-PA9-Pad42)
- U1 pad 43: (no net) -> unconnected-(U1-PA10-Pad43)
- U1 pad 44: (no net) -> unconnected-(U1-PA11-Pad44)
- U1 pad 45: (no net) -> unconnected-(U1-PA12-Pad45)
- U1 pad 5: (no net) -> unconnected-(U1-PH0-Pad5)
- U1 pad 50: (no net) -> unconnected-(U1-PA15-Pad50)
- U1 pad 52: (no net) -> unconnected-(U1-PC11-Pad52)
- U1 pad 53: (no net) -> unconnected-(U1-PC12-Pad53)
- U1 pad 54: (no net) -> unconnected-(U1-PD2-Pad54)
- U1 pad 56: (no net) -> unconnected-(U1-PB4-Pad56)
- U1 pad 57: (no net) -> unconnected-(U1-PB5-Pad57)
- U1 pad 58: (no net) -> unconnected-(U1-PB6-Pad58)
- U1 pad 59: (no net) -> unconnected-(U1-PB7-Pad59)
- U1 pad 6: (no net) -> unconnected-(U1-PH1-Pad6)
- U1 pad 8: (no net) -> unconnected-(U1-PC0-Pad8)
- U1 pad 9: (no net) -> unconnected-(U1-PC1-Pad9)
- U6 pad 1: (no net) -> unconnected-(U6-RS485/GPIO.1-Pad1)
- U6 pad 10: (no net) -> unconnected-(U6-NC-Pad10)
- U6 pad 11: (no net) -> unconnected-(U6-~{SUSPEND}-Pad11)
- U6 pad 13: (no net) -> unconnected-(U6-~{WAKEUP}-Pad13)
- U6 pad 14: (no net) -> unconnected-(U6-SUSPEND-Pad14)
- U6 pad 15: (no net) -> unconnected-(U6-~{CTS}-Pad15)
- U6 pad 16: (no net) -> unconnected-(U6-~{RTS}-Pad16)
- U6 pad 19: (no net) -> unconnected-(U6-~{RXT}/GPIO.3-Pad19)
- U6 pad 2: (no net) -> unconnected-(U6-CLK/GPIO.0-Pad2)
- U6 pad 20: (no net) -> unconnected-(U6-~{TXT}/GPIO.2-Pad20)
