File: Hardware/Rev2_Controller/OSBAMS_Rev2_RELEASE_CANDIDATE_1/probe/01_Probe.kicad_sch (KiCad schematic)
At the start: 5 parts, among them J1 TO_CONTROLLER, U1 TC74A5-3.3VAT

Commit message: RC1: reconcile user-relayed manufacturer data (USER_RELAYED_MANUFACTURER)
- audit report MANUFACTURER_DATA_RECONCILIATION.md; INA228/STM32/IRLML0060/LMR14006Y/CP2102N/VO610A/TC74 pin maps match the relayed data
- ISO7721 pin-direction conflict left unresolved (needs the TI pin diagram); CP2102N VBUS reference connection open
- LMR14006Y: 95 ns TON_MIN analysis (15 V marginal, 24.4 V below TON_MIN); 1.5SMBJ48A vs INA228 85 V clamp-vs-current analysis
- firmware: INA228 IMAX 30 A -> 20 A (SHUNT_CAL 1250) + test
- fix: TC74 probe PCB had been left unrouted by the schematic step; re-routed, DRC 0; schematic step no longer rebuilds it

Co-Authored-By: Claude Sonnet 5.5 <noreply@anthropic.com>
Claude-Session: https://claude.ai/code/session_01HV1TCrYnLTcNjmYdFqCPLo
Parts:
- U1: Evidence UNVERIFIED -> USER_RELAYED_MANUFACTURER
