File: Hardware/Rev2_Controller/rc1_3/OSBAMS_Rev2_RC13/03_MCU.kicad_sch (KiCad schematic)
At the start: 16 parts, among them J9 SWD, SW1 RESET, U1 STM32L476RGT6

Commit message: Controller RC1.3: exact Samtec FTSH-105-01-L-DV-K footprint (drawing rev H), verified 1.5SMBJ12CA data, rerouted; checks clean
Co-Authored-By: Claude Sonnet 5.5 <noreply@anthropic.com>
Claude-Session: https://claude.ai/code/session_01ENatZXrEDA18PaxUrZWrpi
Parts:
- J9: footprint Connector_PinHeader_1.27mm:PinHeader_2x05_P1.27mm_Vertical_SMD -> OSBAMS_Rev2:FTSH-105-01-L-DV-K
