File: Hardware/Rev2_Controller/rc1_3/OSBAMS_Rev2_RC13/05_INA228_Shunt.kicad_sch (KiCad schematic)
At the start: 20 parts, among them J5 SHUNT_KELVIN, U2 INA228

Commit message: Controller RC1.3: exact Samtec FTSH-105-01-L-DV-K footprint (drawing rev H), verified 1.5SMBJ12CA data, rerouted; checks clean
Co-Authored-By: Claude Sonnet 5.5 <noreply@anthropic.com>
Claude-Session: https://claude.ai/code/session_01ENatZXrEDA18PaxUrZWrpi
Parts:
- D20: Evidence UNVERIFIED -> USER_RELAYED_MANUFACTURER
